Commit message: Update SDF.

File: sdf/simplebot/simplebot.urdf (robot description, URDF)
Before this commit: robot myrobot, 1 links, 0 joints
Links:
- link base_link: geometry collision cylinder length=0.6 radius=0.2; visual cylinder length=0.6 radius=0.2

File: sdf/simplebot/simplebot.xacro (robot description, xacro)
@@ -1,4 +1,4 @@
 <?xml version="1.0"?>
-<robot name="myrobot" xmlns:xacro="http://ros.org/wiki/xacro">
+<robot name="simplebot" xmlns:xacro="http://ros.org/wiki/xacro">
   <xacro:property name="the_length" value="0.6" />
   <xacro:property name="the_radius" value="0.2" />
